Commit message: fix

File: urdf/cibo.urdf (robot description, URDF)
Before this commit: robot cibo, 3 links, 2 joints
Links:
- added link base_link
Joints:
- added joint base_pedestal_joint: type fixed, parent base_link, child pedestal_link, origin xyz=0.0 0.0 0.025 rpy=0 0 0

Commit message: fix

File: urdf/cibo.urdf (robot description, URDF)
Before this commit: robot cibo, 4 links, 3 joints
Links:
- added link camera_01_link; visual box size=0.0123 0.0653 0.0225
- added link camera_02_link; visual box size=0.0123 0.0653 0.0225
Joints:
- added joint camera_01_joint: type fixed, parent vertical_bar_link, child camera_01_link, origin xyz=0.025 0.0 0.0 rpy=0 0 0
- added joint camera_02_joint: type fixed, parent horizontal_bar_link, child camera_02_link, origin xyz=0.025 0.0 0.2 rpy=0 1.57 0

Commit message: fix

File: urdf/cibo.urdf (robot description, URDF)
Before this commit: robot cibo, 6 links, 5 joints
Joints:
- joint camera_02_joint: origin xyz=0.025 0.0 0.2 rpy=0 1.57 0 -> xyz=0.025 0.0 0.2 rpy=0 0 0

Commit message: fix

File: urdf/cibo.urdf (robot description, URDF)
Before this commit: robot cibo, 6 links, 5 joints
Links:
- added link map
- link horizontal_bar_link: geometry visual box size=0.025 0.05 0.48
- link pedestal_link: geometry visual box size=0.36 0.36 0.005
- link vertical_bar_link: geometry visual box size=0.025 0.05 0.758
Joints:
- added joint map_base_joint: type fixed, parent map, child base_link
- joint base_pedestal_joint: origin xyz=0.0 0.0 0.025 rpy=0 0 0 -> xyz=0.0 0.0 0.067 rpy=0 0 0
- joint camera_01_joint: origin xyz=0.025 0.0 0.0 rpy=0 0 0 -> xyz=0.025 0.0 -0.311 rpy=0 0 0
- joint pedestal_vertical_joint: origin xyz=-0.1 0.0 0.3 rpy=0 0 0 -> xyz=-0.1 0.0 0.379 rpy=0 0 0
- joint vertical_horizontal_joint: origin xyz=0.2 0.0 0.3 rpy=0 1.57 0 -> xyz=0.2 0.0 0.379 rpy=0 1.57 0

Commit message: fix

File: urdf/cibo.urdf (robot description, URDF)
Before this commit: robot cibo, 7 links, 6 joints
Joints:
- joint camera_02_joint: origin xyz=0.025 0.0 0.2 rpy=0 0 0 -> xyz=0.025 0.0 0.2 rpy=-3.14 0 0

Commit message: fix

File: urdf/cibo.urdf (robot description, URDF)
Before this commit: robot cibo, 7 links, 6 joints
Joints:
- joint camera_01_joint: origin xyz=0.025 0.0 -0.311 rpy=0 0 0 -> xyz=0.16 0.0 -0.311 rpy=0 0 0
